File: mrf24j40-nucleo.kicad_pcb (KiCad board)
At the start: 2 copper layers, 28.6 x 25.4 mm, 2 parts, among them M1 MRF24J40MA_TRANSEIVER_MODULE, P1 CONN_02X08

Commit message: Add name
Other:
- board text added: "Nucleo Keppeltje"
Changed lines of the file:
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@@
     (area 185.344999 83.744999 214.070001 109.295001)
     (thickness 1.6)
-    (drawings 14)
+    (drawings 15)
     (tracks 55)
     (zones 0)
@@
     (0 F.Cu signal)
     (31 B.Cu signal)
-    (32 B.Adhes user hide)
-    (33 F.Adhes user hide)
-    (34 B.Paste user hide)
-    (35 F.Paste user hide)
+    (34 B.Paste user)
+    (35 F.Paste user)
     (36 B.SilkS user)
     (37 F.SilkS user)
     (38 B.Mask user)
     (39 F.Mask user)
-    (40 Dwgs.User user)
-    (41 Cmts.User user)
-    (42 Eco1.User user)
-    (43 Eco2.User user)
     (44 Edge.Cuts user)
-    (45 Margin user)
-    (46 B.CrtYd user)
     (47 F.CrtYd user)
     (48 B.Fab user)
@@
     (descr "Through hole straight pin header, 2x08, 2.54mm pitch, double rows")
     (tags "Through hole pin header THT 2x08 2.54mm double row")
-    (fp_text reference P1 (at 1.27 -2.39) (layer F.SilkS)
+    (fp_text reference P1 (at 1.27 -2.39) (layer F.SilkS) hide
       (effects (font (size 1 1) (thickness 0.15)))
     )
@@
     )
   )
+  (gr_text "Nucleo Keppeltje\n" (at 193.04 85.725) (layer F.SilkS)
+    (effects (font (size 1 1) (thickness 0.25)))
+  )
   (gr_text VCC (at 194.31 104.14) (layer F.SilkS)
     (effects (font (size 0.5 0.5) (thickness 0.125)))
@@
   (via (at 209.55 107.315) (size 0.6) (drill 0.4) (layers F.Cu B.Cu) (net 1))
   (segment (start 209.55 105.41) (end 209.55 107.315) (width 0.25) (layer F.Cu) (net 1))
+  (segment (start 186.69 86.995) (end 186.69 101.6) (width 0.25) (layer F.Cu) (net 2))
   (segment (start 186.69 101.6) (end 189.23 104.14) (width 0.25) (layer B.Cu) (net 2))
   (via (at 186.69 101.6) (size 0.6) (drill 0.4) (layers F.Cu B.Cu) (net 2))
@@
   (segment (start 209.55 85.725) (end 208.28 84.455) (width 0.25) (layer F.Cu) (net 2))
   (segment (start 189.23 84.455) (end 186.69 86.995) (width 0.25) (layer F.Cu) (net 2))
-  (segment (start 186.69 86.995) (end 186.69 101.6) (width 0.25) (layer F.Cu) (net 2))
   (segment (start 204.47 86.36) (end 204.47 87.63) (width 0.25) (layer F.Cu) (net 4))
   (segment (start 203.2 85.09) (end 204.47 86.36) (width 0.25) (layer F.Cu) (net 4))

Commit message: Change sheet size
Parts:
- moved M1 114.7 mm to (95.6, 35.6)
- moved P1 114.7 mm to (87.0, 36.8)
