File: mrf24j40-nucleo.kicad_pcb (KiCad board)
At the start: 2 copper layers, 28.6 x 25.4 mm, 2 parts, among them M1 MRF24J40MA_TRANSEIVER_MODULE, P1 CONN_02X08

Commit message: Reroute
Routing:
- net CS: track 15.0 -> 15.5 mm
Other:
- board text added: "v1.2"
- board text removed: "v1.1"
Changed lines of the file:
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@@
     (thickness 1.6)
     (drawings 14)
-    (tracks 54)
+    (tracks 55)
     (zones 0)
     (modules 2)
@@
     (effects (font (size 1 1) (thickness 0.25)))
   )
-  (gr_text v1.1 (at 100.33 33.655) (layer F.SilkS)
+  (gr_text v1.2 (at 100.33 33.655) (layer F.SilkS)
     (effects (font (size 1 1) (thickness 0.25)))
   )
@@
   (segment (start 90.805 36.83) (end 92.71 38.735) (width 0.25) (layer B.Cu) (net 7))
   (segment (start 89.535 36.83) (end 90.805 36.83) (width 0.25) (layer B.Cu) (net 7))
-  (segment (start 98.425 55.88) (end 99.06 55.245) (width 0.25) (layer B.Cu) (net 8))
-  (segment (start 88.265 55.88) (end 98.425 55.88) (width 0.25) (layer B.Cu) (net 8))
-  (segment (start 88.265 55.88) (end 86.995 54.61) (width 0.25) (layer B.Cu) (net 8))
-  (via (at 99.06 55.245) (size 0.6) (drill 0.4) (layers F.Cu B.Cu) (net 8))
+  (segment (start 91.44 53.34) (end 88.265 53.34) (width 0.25) (layer B.Cu) (net 8))
+  (segment (start 88.265 53.34) (end 86.995 54.61) (width 0.25) (layer B.Cu) (net 8))
+  (via (at 91.44 53.34) (size 0.6) (drill 0.4) (layers F.Cu B.Cu) (net 8))
+  (segment (start 93.345 55.245) (end 91.44 53.34) (width 0.25) (layer F.Cu) (net 8))
+  (segment (start 99.06 55.245) (end 93.345 55.245) (width 0.25) (layer F.Cu) (net 8))
   (segment (start 99.695 54.61) (end 99.06 55.245) (width 0.25) (layer F.Cu) (net 8))
   (segment (start 99.695 53.34) (end 99.695 54.61) (width 0.25) (layer F.Cu) (net 8))
